Commit message: add new tag for skin, change to 100 and 101

File: urdf/aircraft_skin_with_marker.urdf (robot description, URDF)
Before this commit: robot aircraft_skin, 4 links, 3 joints
Links:
- removed link tag36_11_00233
- added link tag36_11_00100; visual mesh filename=package://gerard_bauzil/meshes/apriltag_36h11/tag36_11_0010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 scale=0.0573 0.0573 1.
- added link tag36_11_00101; visual mesh filename=package://gerard_bauzil/meshes/apriltag_36h11/tag36_11_0010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 scale=0.0573 0.0573 1.
Joints:
- added joint to_tag_2: type fixed, parent hole_link, child tag36_11_00101, origin xyz=-0.145 0 0
- joint to_tag: child tag36_11_00233 -> tag36_11_00100; origin xyz=-0.20 0 0 -> xyz=-0.252 0 0
