Commit message: Update with tables

File: urdf/box_with_qr.urdf (robot description, URDF)
Before this commit: robot box, 2 links, 1 joints
Joints:
- joint to_tag: origin xyz=0.05 0 0 -> xyz=0.09 0 0

Commit message: Some update

File: urdf/box_with_qr.urdf (robot description, URDF)
Before this commit: robot box, 2 links, 1 joints
Links:
- removed link base_link
- removed link tag36_11
Joints:
- removed joint to_tag
